File: 64dd/64dd.sch (KiCad schematic (older format))
At the start: 10 parts, among them U201 SD29L, U301 HD153031F, U401 H8329x-FP64, U901 NUD-JPN-2

Commit message: Finished the symbols mostly and traced out the H8
Parts:
- added C414: C_Small, symbol Device:C_Small
- added Jp502: Conn_01x12, symbol Connector_Generic:Conn_01x12
- added P501: Conn_01x11, symbol Connector_Generic:Conn_01x11
- added Q601: Q_NMOS_GDS, symbol Device:Q_NMOS_GDS
- added R212: 51, symbol Device:R_Small
- added R401: 22K, symbol Device:R_Small
- added R403: 2.2K, symbol Device:R_Small
- added R405, R417, R419: 10K, symbol Device:R_Small
- added R418: 15K, symbol Device:R_Small
- added R603: 33K, symbol Device:R_Small
- added U402: MC33174, symbol Amplifier_Operational:MC33174
- added U403: C46T6, symbol 64dd:C46T6
- added U404: JRC2103, symbol 64dd:JRC2103
- added U409: RTC-4543, symbol 64dd:RTC-4543
- added U?: BA6832FS, symbol 64dd:BA6832FS
- R409, R410, R412, R413: value ? -> 10K
Connections:
- net labels added: +5V, GND
- wire segments 38 -> 198
- no-connect marks 0 -> 29
Other:
- note added: "NOTE: There are filter inductors on the +5V net not shown"
- note added: "x16 Mode"
- moved on the sheet: R310, R319, R409, R410, R412, R413

Commit message: Mapped out the connectivity to the heads
Parts:
- added C323, C324: C_Small, symbol Device:C_Small
- added R208: 18K, symbol Device:R_Small
- added R209: 8.2K, symbol Device:R_Small
- added R423: 2.2K, symbol Device:R_Small
Connections:
- net +5V: now also R423.2
- net GND: now also R208.1
- net at Jp502.4 (Pin_4), U401.4 (~RES~), U404.8 (~RESET~): now also R209.1, R423.1
- net at U301.85 (RINX): now also C324.1
- net at U301.86 (RINY): now also C323.1
- net at U201.64: now also Jp502.8 (Pin_8)
- net at U201.65: now also Jp502.5 (Pin_5)
- net at U201.83: now also R208.2, R209.2
- net at Jp502.6 (Pin_6): now also C323.2
- net at Jp502.7 (Pin_7): now also C324.2
Other:
- note added: "Endstop Microswitch?"
- note added: "Head Select"
- note added: "R/~W~ Select"
Changed lines of the file:
@@
 Sheet 1 1
 Title "64DD JPN Retail Schematics"
-Date "2020-08-15"
-Rev "0"
+Date "2020-08-20"
+Rev "1"
 Comp "@ChrisPVille"
 Comment1 ""
@@
 	31500 10450 31500 10650
 Connection ~ 31950 17550
+$Comp
+L Device:R_Small R209
+U 1 1 5F3B2D13
+P 22700 16450
+F 0 "R209" V 22625 16450 39  0000 C CNN
+F 1 "8.2K" V 22700 16450 39  0000 C CNN
+F 2 "" H 22700 16450 50  0001 C CNN
+F 3 "~" H 22700 16450 50  0001 C CNN
+	1    22700 16450
+	0    1    1    0
+$EndComp
+Wire Wire Line
+	29550 15750 29550 17200
+Wire Wire Line
+	29550 17200 23050 17200
+Wire Wire Line
+	23050 17200 23050 16450
+Wire Wire Line
+	23050 16450 22800 16450
+Connection ~ 29550 15750
+Wire Wire Line
+	22600 16450 22400 16450
+Wire Wire Line
+	22400 16450 22400 16150
+Wire Wire Line
+	22400 16150 17100 16150
+$Comp
+L Device:R_Small R208
+U 1 1 5F3D69A3
+P 22400 16600
+F 0 "R208" V 22325 16600 39  0000 C CNN
+F 1 "18K" V 22400 16600 39  0000 C CNN
+F 2 "" H 22400 16600 50  0001 C CNN
+F 3 "~" H 22400 16600 50  0001 C CNN
+	1    22400 16600
+	-1   0    0    1
+$EndComp
+Wire Wire Line
+	22400 16500 22400 16450
+Connection ~ 22400 16450
+$Comp
+L power:GND #PWR?
+U 1 1 5F3E378A
+P 22400 16700
+F 0 "#PWR?" H 22400 16450 50  0001 C CNN
+F 1 "GND" H 22405 16527 50  0000 C CNN
+F 2 "" H 22400 16700 50  0001 C CNN
+F 3 "" H 22400 16700 50  0001 C CNN
+	1    22400 16700
+	1    0    0    -1
+$EndComp
+Text Notes 26100 12950 1    50   ~ 0
+Endstop Microswitch?
+$Comp
+L Device:C_Small C324
+U 1 1 5F3E65F7
+P 14350 4350
+F 0 "C324" V 14475 4250 50  0000 L CNN
+F 1 "C_Small" H 14442 4305 50  0001 L CNN
+F 2 "" H 14350 4350 50  0001 C CNN
+F 3 "~" H 14350 4350 50  0001 C CNN
+	1    14350 4350
+	0    1    1    0
+$EndComp
+$Comp
+L Device:C_Small C323
+U 1 1 5F3E7B66
+P 14350 4650
+F 0 "C323" V 14475 4550 50  0000 L CNN
+F 1 "C_Small" H 14442 4605 50  0001 L CNN
+F 2 "" H 14350 4650 50  0001 C CNN
+F 3 "~" H 14350 4650 50  0001 C CNN
+	1    14350 4650
+	0    1    1    0
+$EndComp
+Wire Wire Line
+	15400 4450 14700 4450
+Wire Wire Line
+	14700 4450 14700 4350
+Wire Wire Line
+	14700 4350 14450 4350
+Wire Wire Line
+	14450 4650 14700 4650
+Wire Wire Line
+	14700 4650 14700 4550
+Wire Wire Line
+	14700 4550 15400 4550
+Wire Wire Line
+	14250 4350 11800 4350
+Wire Wire Line
+	11800 4350 11800 4900
+Wire Wire Line
+	14250 4650 11900 4650
+Wire Wire Line
+	11900 4650 11900 5000
+$Comp
+L Device:R_Small R423
+U 1 1 5F44986F
+P 29350 10550
+F 0 "R423" V 29275 10550 39  0000 C CNN
+F 1 "2.2K" V 29350 10550 39  0000 C CNN
+F 2 "" H 29350 10550 50  0001 C CNN
+F 3 "~" H 29350 10550 50  0001 C CNN
+	1    29350 10550
+	0    1    1    0
+$EndComp
+$Comp
+L power:+5V #PWR?
+U 1 1 5F44B602
+P 29200 10500
+F 0 "#PWR?" H 29200 10350 50  0001 C CNN
+F 1 "+5V" V 29215 10628 50  0000 L CNN
+F 2 "" H 29200 10500 50  0001 C CNN
+F 3 "" H 29200 10500 50  0001 C CNN
+	1    29200 10500
+	1    0    0    -1
+$EndComp
+Wire Wire Line
+	29200 10500 29200 10550
+Wire Wire Line
+	29200 10550 29250 10550
+Wire Wire Line
+	29450 10550 29550 10550
+Wire Wire Line
+	10750 4900 10750 4350
+Wire Wire Line
+	10750 4900 11800 4900
+Wire Wire Line
+	10850 4350 10850 5000
+Wire Wire Line
+	10850 5000 11900 5000
+Wire Wire Line
+	10950 4350 10950 8950
+Wire Wire Line
+	10950 8950 4950 8950
+Wire Wire Line
+	4950 8950 4950 19050
+Wire Wire Line
+	4950 19050 15200 19050
+Wire Wire Line
+	15200 19050 15200 16700
+Wire Wire Line
+	10650 4350 10650 8850
+Wire Wire Line
+	10650 8850 4850 8850
+Wire Wire Line
+	4850 8850 4850 19150
+Wire Wire Line
+	4850 19150 15100 19150
+Wire Wire Line
+	15100 19150 15100 16700
+Wire Wire Line
+	11250 4350 11250 4450
+Wire Wire Line
+	10250 4350 10250 4450
+Text Notes 10600 5550 1    50   ~ 0
+Head Select
+Text Notes 10900 5550 1    50   ~ 0
+R/~W~ Select
 $EndSCHEMATC
